Commit message: backup

File: steer_drive/cirkit_unit03_description/urdf/cirkit_unit03.xacro (robot description, xacro)
@@ -39,5 +39,5 @@
       <origin rpy="0 0 0" xyz="0 0 0"/>
       <geometry>
-        <mesh filename="package://cirkit_unit03_description/meshes/LRF/UTM-30LX.dae"/>
+        <mesh filename="package://cirkit_unit03_description/meshes/LRF/UTM-30LX.dae"/> <!-- mesh do LIDAR -->
       </geometry>
     </visual>
@@ -54,5 +54,5 @@
       <origin rpy="0 0 0" xyz="0 0 0"/>
       <geometry>
-        <mesh filename="package://cirkit_unit03_description/meshes/LRF/UTM-30LX.dae"/>
+        <mesh filename="package://cirkit_unit03_description/meshes/LRF/UTM-30LX.dae"/> <!-- mesh do LIDAR -->
       </geometry>
     </visual>

Commit message: params set

File: steer_drive/cirkit_unit03_description/urdf/cirkit_unit03.xacro (robot description, xacro)
@@ -24,5 +24,11 @@
       <origin rpy="0 0 0" xyz="0 0 0.9" />
       <geometry>
-        <box size="2.5 0.8 0.8"/>
+        <box size="2.5 1 0.5657"/>
+      </geometry>
+    </collision>
+    <collision>
+      <origin rpy="0 0 0.785" xyz="1.25 0 0.9" />
+      <geometry>
+        <box size="0.5657 0.5657 0.5657"/>
       </geometry>
     </collision>

Commit message: collision model placed

File: steer_drive/cirkit_unit03_description/urdf/cirkit_unit03.xacro (robot description, xacro)
@@ -14,5 +14,5 @@
     <visual>
       <!-- <origin rpy="0 0 0" xyz="0 0 0.55" /> -->
-      <origin xyz="-1.7575 -0.91 0.05" rpy="${PI/2} 0.02 ${PI/2}"/>
+      <origin xyz="-1.7575 -0.91 0.05" rpy="${PI/2} 0 ${PI/2}"/>
       <geometry>
         <!-- <mesh filename="package://cirkit_unit03_description/meshes/cirkit_unit03/cirkit_unit03_body.dae"/> -->
@@ -22,13 +22,16 @@
     </visual>
     <collision>
-      <origin rpy="0 0 0" xyz="0 0 0.9" />
+      <origin rpy="${PI/2} 0 0" xyz="-0.9 0.7 0.5" />
+      <!-- <origin xyz="-1.7575 -0.91 0.05" rpy="${PI/2} 0.02 ${PI/2}"/> -->
       <geometry>
-        <box size="2.5 1 0.5657"/>
+        <!-- <box size="2.24 1.4 0.5657"/> -->
+        <mesh filename="package://cirkit_unit03_description/meshes/cirkit_unit03/collision_small.STL" scale="0.001 0.001 0.001"/>
       </geometry>
     </collision>
     <collision>
-      <origin rpy="0 0 0.785" xyz="1.25 0 0.9" />
+      <origin rpy="0 0 0" xyz="-0.882946311 0 0.78285" />
+      <!-- <origin xyz="-1.7575 -0.91 0.05" rpy="${PI/2} 0.02 ${PI/2}"/> -->
       <geometry>
-        <box size="0.5657 0.5657 0.5657"/>
+        <box size="1.6 1.4 0.5657"/>
       </geometry>
     </collision>
@@ -45,5 +48,6 @@
       <origin rpy="0 0 0" xyz="0 0 0"/>
       <geometry>
-        <mesh filename="package://cirkit_unit03_description/meshes/LRF/UTM-30LX.dae"/> <!-- mesh do LIDAR -->
+        <mesh filename="package://cirkit_unit03_description/meshes/LRF/UTM-30LX.dae"/>
+        <!-- mesh do LIDAR -->
       </geometry>
     </visual>
@@ -60,5 +64,6 @@
       <origin rpy="0 0 0" xyz="0 0 0"/>
       <geometry>
-        <mesh filename="package://cirkit_unit03_description/meshes/LRF/UTM-30LX.dae"/> <!-- mesh do LIDAR -->
+        <mesh filename="package://cirkit_unit03_description/meshes/LRF/UTM-30LX.dae"/>
+        <!-- mesh do LIDAR -->
       </geometry>
     </visual>
